File: dce-pcb-v1/dce-pcb-v1.kicad_pcb (KiCad board)
At the start: 2 copper layers, 42 parts, among them J1 Conn_01x05_Socket, M1 2N7000, Q1 BC557B, Q10 BC547B, Q11 BC547B, Q2 BC557B, Q3 BC547B, Q4 BC547B, Q5 TIP42C, Q6 TIP41C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

Commit message: actualiza el pcb
Parts:
- renumbered Q11 to Q5, Q10 to Q6, Q6 to Q8, Q5 to Q9, R23 to R1, R25 to R10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
