File: dce-pcb-v1/dce-pcb-v1.kicad_sch (KiCad schematic)
At the start: 42 parts, among them J1 Conn_01x05_Socket, M1 2N7000, Q1 BC557B, Q10 BC547B, Q11 BC547B, Q2 BC557B, Q3 BC547B, Q4 BC547B, Q5 TIP42C, Q6 TIP41C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

Commit message: actualiza el pcb
Parts:
- removed RL1: RL, Resistor_THT:R_Axial_DIN0207_L6.3mm_D2.5mm_P7.62mm_Horizontal, symbol ltspice:res
- J1: symbol Connector:Conn_01x05_Socket -> Connector:Conn_01x06_Socket
Connections:
- net Vo: now also J1.6 (Pin_6)
Other:
- moved on the sheet: R13, R14, R15, R16, R17, R18, R19, R20, R24, U5A, U5B, U5C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
