File: Checkpoint 2/DCE - PCB - v1/dce-pcb-v1.kicad_pcb (KiCad board)
At the start: 2 copper layers, 42 parts, among them J1 Conn_01x05_Socket, M1 2N7000, Q1 BC557B, Q2 BC557B, Q3 BC547B, Q4 BC547B, Q5 BC547B, Q6 BC547B, Q7 BC547B, Q8 TIP41C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

Commit message: Sube esquematico y diseño del pcb actualizados
Falta organizar el pcb
Parts:
- removed R24: 4.7k, Resistor_THT:R_Axial_DIN0207_L6.3mm_D2.5mm_P7.62mm_Horizontal
- removed R25: 100, Resistor_THT:R_Axial_DIN0207_L6.3mm_D2.5mm_P7.62mm_Horizontal
- removed RL1: RL, Resistor_THT:R_Axial_DIN0207_L6.3mm_D2.5mm_P7.62mm_Horizontal
- removed U2: LM324, Package_DIP:DIP-14_W7.62mm_Socket
- added C1: 2.2n, Capacitor_THT:C_Disc_D3.4mm_W2.1mm_P2.50mm, F.Cu at (155.4, 51.2)
- added C3: 100p, Capacitor_THT:C_Disc_D3.4mm_W2.1mm_P2.50mm, F.Cu at (155.4, 54.9)
- added C4: 10u, Capacitor_THT:C_Disc_D3.4mm_W2.1mm_P2.50mm, F.Cu at (155.4, 58.5)
- added C5: 10u, Capacitor_THT:C_Disc_D3.4mm_W2.1mm_P2.50mm, F.Cu at (155.4, 62.1)
- added C6: 10u, Capacitor_THT:C_Disc_D3.4mm_W2.1mm_P2.50mm, F.Cu at (155.4, 65.8)
- added C7: 10u, Capacitor_THT:C_Disc_D3.4mm_W2.1mm_P2.50mm, F.Cu at (155.4, 69.5)
- added C8: 10u, Capacitor_THT:C_Disc_D3.4mm_W2.1mm_P2.50mm, F.Cu at (155.4, 73.1)
- added J2: Conn_01x02_Socket, TerminalBlock_4Ucon:TerminalBlock_4Ucon_1x02_P3.50mm_Horizontal, F.Cu at (147.2, 83.5)
- added Rcp1: 470, Resistor_THT:R_Axial_DIN0207_L6.3mm_D2.5mm_P7.62mm_Horizontal, F.Cu at (144.6, 71.7)
- added TP1: TestPoint, TestPoint:TestPoint_THTPad_1.0x1.0mm_Drill0.5mm, F.Cu at (172.7, 50.9)
- added TP2: TestPoint, TestPoint:TestPoint_THTPad_1.0x1.0mm_Drill0.5mm, F.Cu at (172.7, 54.0)
- added TP3: TestPoint, TestPoint:TestPoint_THTPad_1.0x1.0mm_Drill0.5mm, F.Cu at (172.7, 57.0)
- added TP4: TestPoint, TestPoint:TestPoint_THTPad_1.0x1.0mm_Drill0.5mm, F.Cu at (172.7, 60.0)
- J1: value Conn_01x05_Socket -> Conn_01x06_Socket; footprint Connector_PinSocket_1.00mm:PinSocket_1x05_P1.00mm_Vertical -> TerminalBlock_4Ucon:TerminalBlock_4Ucon_1x06_P3.50mm_Horizontal
- Q1, Q2: value BC557B -> BC547B
- Q4, Q5: value BC547B -> BC557B
- Q7: value BC547B -> TIP41C
- Q8: value TIP41C -> TIP42C
- Q9: value TIP42C -> BC547B; footprint Package_TO_SOT_THT:TO-220-3_Vertical -> Package_TO_SOT_THT:TO-92L_Inline
- R1: value 2.7k -> 3.3k
- R10, R9: value 10k -> 1.5k
- R11: value 1k -> 2.7k
- R12: value 100k -> 390
- R13: value 1k -> 1K
- R14: value 100k -> 680
- R15: value 1k -> 270
- R16: value 1.5k -> 100
- R17, R22: value 1.5k -> 1k
- R18: value 1.5k -> 100k
- R19: value 1.5k -> 10k
- R2: value 390 -> 5.6k
- R20: value 6.8k -> 1k
- R21: value 8.2k -> 1.5k
- R23: value 2.7k -> 10k
- R3: value 1K -> 6.8k
- R4: value 680 -> 1.2k
- R5: value 270 -> 2.7k
- R6: value 3.3k -> 1.5k
- R7: value 1k -> 6.8k
- R8: value 1k -> 510
- moved J1 59.8 mm to (124.6, 94.3)
- moved Q9 48.0 mm to (169.0, 89.5)
- moved R21 43.9 mm to (144.6, 51.4)
- moved RE1 42.2 mm to (144.6, 63.5)
- moved R12 37.3 mm to (133.8, 55.5)
- moved U1 37.3 mm to (161.5, 51.5)
- moved R1 35.9 mm to (123.0, 51.4)
- moved Rs1 35.3 mm to (144.6, 75.7)
- moved R10 35.3 mm to (123.0, 87.8)
- moved R22 34.0 mm to (144.6, 55.5)
- moved R23 31.7 mm to (144.6, 59.5)
- moved R11 28.7 mm to (133.8, 51.4)
- moved R20 26.7 mm to (133.8, 87.8)
- moved R13 26.4 mm to (133.8, 59.5)
- moved R7 25.8 mm to (123.0, 75.7)
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Connections:
- J1 pad 2: /VPOSA -> /-VPOSA
- J1 pad 3: /Vref -> /+VPOSA
- J1 pad 4: /Vreg -> /Vref
- J1 pad 5: /Vsel -> /Vreg
- Q1 pad 3: Net-(Q1-E) -> 0
- Q2 pad 1: /Vlc -> Net-(Q2-C)
- Q2 pad 2: Net-(Q1-B) -> /Vref
- Q3 pad 1: Net-(Q1-B) -> Net-(Q2-E)
- Q3 pad 2: /Vref -> Net-(Q1-B)
- Q3 pad 3: Net-(Q3-E) -> 0
- Q4 pad 1: /Vlc -> Net-(Q2-C)
- Q4 pad 2: /Vf -> Net-(Q2-C)
- Q4 pad 3: Net-(Q3-E) -> Net-(Q4-E)
- Q5 pad 1: Net-(Q5-B) -> /Vlc
- Q5 pad 2: Net-(Q5-B) -> Net-(Q2-C)
- Q5 pad 3: 0 -> Net-(Q5-E)
- Q6 pad 1: Net-(Q3-E) -> /Vlc
- Q6 pad 2: Net-(Q5-B) -> /Vf
- Q6 pad 3: 0 -> Net-(Q2-E)
- Q7 pad 1: /Vlc -> Net-(Q7-C)
- Q7 pad 2: Net-(Q7-B) -> /Vlc
- Q8 pad 1: Net-(Q8-C) -> Net-(Q7-E)
- Q8 pad 2: /Vlc -> Net-(Q7-C)
- Q8 pad 3: Net-(Q8-E) -> /Vreg
- Q9 pad 1: Net-(Q8-E) -> /Vlc
- Q9 pad 2: Net-(Q8-C) -> Net-(Q9-B)
- Q9 pad 3: /Vreg -> Net-(Q9-E)
- R1 pad 1: Net-(Q8-E) -> /Vreg
- R1 pad 2: Net-(R1-Pad2) -> Net-(Q1-B)
- R10 pad 1: Net-(U2A--) -> /Sum
- R10 pad 2: Net-(R10-Pad2) -> Net-(U1A--)
- R11 pad 1: Net-(R10-Pad2) -> Net-(Q7-E)
- R12 pad 2: 0 -> /Vf
- R13 pad 1: /vref-c -> /Vf
- R13 pad 2: Net-(U2B--) -> Net-(M1-D)
- R14 pad 1: Net-(U2B--) -> Net-(M1-D)
- R15 pad 2: Net-(Q7-B) -> 0
- R16 pad 1: /vref-c -> Net-(Q9-E)
- R16 pad 2: Net-(U1C--) -> 0
- R17 pad 1: Net-(U1C--) -> Net-(R17-Pad1)
- R17 pad 2: 0 -> Net-(Q9-B)
- R18 pad 1: Net-(U1C-+) -> /Sum
- R18 pad 2: Net-(U1A--) -> Net-(R17-Pad1)
- R19 pad 1: Net-(U1C-+) -> Net-(U1D--)
- R19 pad 2: Net-(U1B--) -> Net-(R19-Pad2)
- R2 pad 1: Net-(R1-Pad2) -> Net-(R2-Pad1)
- R2 pad 2: /Vf -> /Vref
- R20 pad 1: Net-(U1B-+) -> Net-(Q7-E)
- R20 pad 2: 0 -> Net-(U1D--)
- R21 pad 1: Net-(U1B-+) -> Net-(R19-Pad2)
- R21 pad 2: /Vf -> /Sum
- R22 pad 1: Net-(U1A-+) -> /Vo
- R22 pad 2: 0 -> Net-(U1D-+)
- R23 pad 1: Net-(U1A-+) -> Net-(U1D-+)
- R23 pad 2: Net-(R23-Pad2) -> 0
- R3 pad 1: /Vf -> Net-(R3-Pad1)
- R3 pad 2: Net-(M1-D) -> /Vf
- R4 pad 1: Net-(M1-D) -> Net-(U1B-+)
- R4 pad 2: Net-(R4-Pad2) -> Net-(R3-Pad1)
- R5 pad 1: Net-(R4-Pad2) -> Net-(U1A-+)
- R5 pad 2: 0 -> Net-(R2-Pad1)
- R6 pad 1: /Vreg -> Net-(U1A-+)
- R6 pad 2: Net-(Q5-B) -> 0
- R7 pad 1: Net-(Q8-E) -> Net-(U1B-+)
- R7 pad 2: Net-(U2A-+) -> Net-(R7-Pad2)
- R8 pad 1: /Vo -> Net-(R7-Pad2)
- R8 pad 2: Net-(U2A--) -> 0
- R9 pad 1: Net-(U2A-+) -> /Sum
- R9 pad 2: 0 -> Net-(U1B--)
- RE1 pad 2: Net-(Q1-E) -> Net-(Q4-E)
- RE2 pad 2: Net-(Q2-E) -> Net-(Q5-E)
- Rs1 pad 2: Net-(Q8-E) -> Net-(Q7-E)
- U1 pad 10: Net-(U1C-+) -> 0
- U1 pad 11: 0 -> /-VPOSA
- U1 pad 13: Net-(U1D-+) -> Net-(U1D--)
- U1 pad 14: Net-(U1D-+) -> Net-(R19-Pad2)
- U1 pad 4: /VPOSA -> /+VPOSA
- U1 pad 8: /vref-c -> Net-(R17-Pad1)
- U1 pad 9: Net-(U1C--) -> /Sum

Commit message: avance pcb
Parts:
- C1, C3, C4, C5, C6, C7, C8: footprint Capacitor_THT:C_Disc_D3.4mm_W2.1mm_P2.50mm -> Capacitor_THT:CP_Radial_D5.0mm_P2.00mm
- moved R3 109.2 mm to (206.2, 130.3)
- moved J1 105.4 mm to (228.5, 76.5), turned to -90 degrees
- moved TP3 101.3 mm to (160.0, 157.5)
- moved R16 99.2 mm to (98.0, 164.2), turned to -90 degrees
- moved R4 97.7 mm to (194.4, 130.3)
- moved Q9 96.4 mm to (98.0, 154.8), turned to -90 degrees
- moved R18 94.0 mm to (172.3, 165.5), turned to 180 degrees
- moved R8 93.8 mm to (190.0, 145.5), turned to -90 degrees
- moved Q4 91.8 mm to (81.5, 40.5), turned to 90 degrees
- moved Q1 90.3 mm to (66.0, 75.3), turned to -90 degrees
- moved R7 89.0 mm to (190.0, 134.3), turned to -90 degrees
- moved R17 84.6 mm to (156.0, 157.3), turned to 180 degrees
- moved Q5 80.9 mm to (98.0, 40.5), turned to 90 degrees
- moved Q2 78.1 mm to (81.5, 65.8), turned to -90 degrees
- moved R2 75.4 mm to (126.3, 130.8), turned to 180 degrees
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
Commit message: avance pcb
Parts:
- moved R2 74.2 mm to (186.5, 87.5), turned to -90 degrees
- moved R5 57.0 mm to (183.0, 95.1), turned to 90 degrees
- moved R6 41.9 mm to (168.7, 98.2)
- moved R8 39.4 mm to (181.0, 107.1), turned to 90 degrees
- moved R3 38.1 mm to (174.0, 110.0), turned to -90 degrees
- moved R7 37.0 mm to (177.5, 99.5)
- moved R4 36.8 mm to (174.0, 99.7), turned to -90 degrees
- moved R9 34.4 mm to (157.4, 102.5)
- moved R10 31.8 mm to (157.4, 99.0), turned to 0 degrees
- moved R21 29.8 mm to (159.0, 87.5)
- moved U1 11.0 mm to (163.8, 95.0)
Routing:
- net Net-(U1B--): track 0.00 -> 40.6 mm
- net Net-(U1A-+): track 0.00 -> 19.6 mm
- net /Sum: track 0.00 -> 8.49 mm
- net Net-(U1B-+): track 0.00 -> 8.29 mm
- net Net-(U1A--): track 0.00 -> 6.58 mm
- net Net-(R19-Pad2): track 0.00 -> 4.85 mm
- net Net-(R7-Pad2): track 0.00 -> 3.50 mm
- net Net-(R2-Pad1): track 0.00 -> 3.50 mm
- net Net-(R3-Pad1): track 0.00 -> 2.69 mm

Commit message: pcb_almost_finished
Parts:
- C1, C3: footprint Capacitor_THT:CP_Radial_D5.0mm_P2.00mm -> Capacitor_THT:C_Disc_D3.4mm_W2.1mm_P2.50mm
- moved R16 111.9 mm to (142.5, 61.5)
- moved Q9 108.1 mm to (142.6, 56.4)
- moved R17 92.5 mm to (147.0, 65.3), turned to 90 degrees
- moved R18 91.0 mm to (147.1, 78.0), turned to 90 degrees
- moved TP3 90.1 mm to (147.1, 68.3)
- moved R1 75.3 mm to (127.0, 71.2)
- moved Q1 65.5 mm to (130.6, 86.3)
- moved Q4 61.5 mm to (131.6, 76.2)
- moved RE1 61.2 mm to (130.8, 63.2)
- moved Q5 52.4 mm to (136.3, 76.2)
- moved Q2 51.2 mm to (130.7, 80.1)
- moved RE2 51.1 mm to (134.0, 63.2)
- moved Q3 46.3 mm to (135.4, 86.3)
- moved Q6 40.2 mm to (135.5, 80.1)
- moved J1 35.7 mm to (193.6, 69.2)
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Routing:
- net /Vreg: track 0.00 -> 132.3 mm
- net /Vref: track 0.00 -> 93.5 mm
- net /+VPOSA: track 0.00 -> 62.7 mm
- net /Vf: track 0.00 -> 48.8 mm
- net Net-(Q7-E): track 0.00 -> 46.2 mm
- net /Vsel: track 0.00 -> 43.7 mm
- net /-VPOSA: track 0.00 -> 38.1 mm
- net /Sum: track 8.49 -> 45.8 mm
- net Net-(R17-Pad1): track 0.00 -> 31.7 mm
- net /Vo: track 0.00 -> 23.1 mm
- net /Vlc: track 0.00 -> 21.7 mm
- net Net-(U1B--): track 40.6 -> 24.1 mm
- net Net-(Q1-B): track 0.00 -> 15.1 mm
- net Net-(U1D-+): track 0.00 -> 13.7 mm
- net Net-(M1-D): track 0.00 -> 13.0 mm
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- added copper zone on B.Cu, net 0
Other:
- board outline added: 190.4 x 110.6 mm

Commit message: Actualizacion PCB
Parts:
- moved Vop 2.60 mm to (149.7, 67.9)
- moved R16 0.82 mm to (143.3, 61.5)
- moved J1 0.60 mm to (194.2, 69.2)
- moved C3 0.52 mm to (140.9, 71.6)
- moved Q8 0.35 mm to (142.7, 52.3)
- moved R11 0.27 mm to (143.9, 71.6)
- moved R14 0.17 mm to (146.9, 81.5)
- renumbered TP4 to GND, TP2 to Vd, TP1 to Vf, TP3 to Vop
Connections:
- C6 pad 1: /Vref -> /Vreg
- C7 pad 1: /Vreg -> /Vref
- J1 pad 4: /Vref -> /Vreg
- J1 pad 5: /Vreg -> /Vref
Routing:
- net /Vref: track 93.5 -> 122.2 mm
- net /Vlc: track 21.7 -> 42.4 mm
- net /Vreg: track 132.3 -> 128.5 mm
- net /Vf: track 48.8 -> 52.6 mm
- net Net-(C1-Pad1): track 0.00 -> 2.92 mm
- net Net-(Q7-E): track 46.2 -> 47.3 mm
- net Net-(R17-Pad1): track 31.7 -> 32.7 mm
Other:
- board outline removed
- board text added: "Circuito LDO 3.3V/5V Grupo 5"
- board text added: "GND Vo"
- board text added: "Vsel Vref Vreg +VP -VP GND"
