File: Checkpoint 2/DCE - PCB - v1/dce-pcb-v1.kicad_pcb (KiCad board)
At the start: 2 copper layers, 51 parts, among them J1 Conn_01x06_Socket, J2 Conn_01x02_Socket, M1 2N7000, Q1 BC547B, Q2 BC547B, Q3 BC547B, Q4 BC557B, Q5 BC557B, Q6 BC547B, Q7 TIP41C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

Commit message: PCB actualizado
Parts:
- added GND: TestPoint, TestPoint:TestPoint_THTPad_1.0x1.0mm_Drill0.5mm, F.Cu at (127.2, 61.5)
- C4, C5, C6, C7, C8: footprint Capacitor_THT:CP_Radial_D5.0mm_P2.00mm -> Capacitor_THT:CP_Radial_D5.0mm_P2.50mm
- M1, Q1, Q2, Q3, Q4, Q5, Q6, Q7, Q9: footprint Package_TO_SOT_THT:TO-92L_Inline -> Package_TO_SOT_THT:TO-92L_Inline_Wide
- moved M1 3.19 mm to (151.8, 84.1)
- moved RE1 2.89 mm to (130.4, 60.3)
- moved RE2 2.89 mm to (133.6, 60.3)
- moved Q7 2.84 mm to (136.2, 49.9)
- moved Q9 2.81 mm to (142.3, 53.5)
- moved R1 1.95 mm to (127.0, 69.2)
- moved Q8 1.70 mm to (142.7, 50.6)
- moved Q3 1.27 mm to (135.5, 87.6)
- moved Q1 1.27 mm to (130.6, 87.6)
- moved R12 0.81 mm to (140.1, 82.3)
- moved R14 0.81 mm to (146.9, 82.3)
- moved R13 0.81 mm to (143.4, 90.0)
- moved Q5 0.75 mm to (136.4, 77.0)
- moved Q4 0.75 mm to (131.6, 77.0)
- moved Rs1 0.70 mm to (160.6, 52.6)
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Routing:
- net /Vref: track 122.2 -> 131.1 mm
- net /Vlc: track 42.4 -> 48.4 mm
- net Net-(Q1-B): track 15.1 -> 19.6 mm
- net Net-(M1-D): track 13.0 -> 9.13 mm
- net /-VPOSA: track 38.1 -> 41.8 mm
- net 0: track 2.77 -> 0.00 mm
- net Net-(Q5-E): track 4.04 -> 6.00 mm
- net /Sum: track 45.8 -> 47.6 mm
- net Net-(Q7-E): track 47.3 -> 49.0 mm
- net /Vo: track 23.1 -> 24.5 mm
- net /Vsel: track 43.7 -> 45.0 mm
- net Net-(Q4-E): track 3.28 -> 4.43 mm
- net Net-(R17-Pad1): track 32.7 -> 33.8 mm
- net /Vf: track 52.6 -> 53.6 mm
- net Net-(R11-Pad2): track 4.73 -> 5.72 mm
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Other:
- board text added: "Circuito 3.3V/5V Grupo 5"
- board text added: "LDO"

Commit message: actualizacion PCB
Parts:
- GND (x2), Vd, Vf, Vop: footprint TestPoint:TestPoint_THTPad_1.0x1.0mm_Drill0.5mm -> LDO_C2:TestPoint_THTPad_1.3x1.3mm_Drill0.7mm
- J1: footprint TerminalBlock_4Ucon:TerminalBlock_4Ucon_1x06_P3.50mm_Horizontal -> LDO_C2:TerminalBlock_4Ucon_1x06_P3.50mm_Horizontal
- J2: footprint TerminalBlock_4Ucon:TerminalBlock_4Ucon_1x02_P3.50mm_Horizontal -> LDO_C2:TerminalBlock_4Ucon_1x02_P3.50mm_Horizontal(3D)
- U1: footprint Package_DIP:DIP-14_W7.62mm_Socket -> LDO_C2:DIP-14_W7.62mm_Socket

Commit message: pcb
Other:
- board outline added: 74.8 x 50.7 mm
Changed lines of the file:
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@@
 		)
 	)
+	(gr_rect
+		(start 123.8 46.2)
+		(end 198.6 96.9)
+		(stroke
+			(width 0.05)
+			(type default)
+		)
+		(fill none)
+		(layer "Edge.Cuts")
+	)
 	(gr_text " LDO "
-		(at 188.75 48.95 0)
+		(at 189.1 49.35 0)
 		(layer "B.Cu")
 		(effects
@@
 	)
 	(gr_text "Circuito\n3.3V/5V\nGrupo 5"
-		(at 197.15 53.8 0)
+		(at 197.5 54.2 0)
 		(layer "B.Cu")
 		(effects
@@
 	)
 	(gr_text "Circuito LDO 3.3V/5V\nGrupo 5"
-		(at 182.5 50.2 0)
+		(at 182.55 50.3 0)
 		(layer "F.SilkS")
 		(effects
@@
 			)
 		)
-	)
-	(zone
-		(net 0)
-		(net_name "")
-		(layer "Edge.Cuts")
-		(hatch edge 0.5)
-		(connect_pads
-			(clearance 0)
-		)
-		(min_thickness 0.25)
-		(filled_areas_thickness no)
-		(keepout
-			(tracks not_allowed)
-			(vias not_allowed)
-			(pads not_allowed)
-			(copperpour allowed)
-			(footprints allowed)
-		)
-		(fill
-			(thermal_gap 0.5)
-			(thermal_bridge_width 0.5)
-		)
-		(polygon
-			(pts
-				(xy 198.6 46.2) (xy 198.6 96.9) (xy 123.8 96.9) (xy 123.8 46.2)
-			)
-		)

Commit message: pcb actualizado con recomendaciones de julio
Parts:
- removed C7, C8: 10u, Capacitor_THT:CP_Radial_D5.0mm_P2.50mm
- added C10: 10n, Capacitor_THT:C_Disc_D3.4mm_W2.1mm_P2.50mm, F.Cu at (190.6, 63.1)
- added C2: 10n, Capacitor_THT:C_Disc_D3.4mm_W2.1mm_P2.50mm, F.Cu at (188.5, 78.7)
- added C9: 10n, Capacitor_THT:C_Disc_D3.4mm_W2.1mm_P2.50mm, F.Cu at (188.4, 75.9)
- added J3: Conn_01x02_Socket, Connector_PinHeader_2.54mm:PinHeader_1x02_P2.54mm_Vertical, F.Cu at (187.8, 87.8)
- Rcp1: value 470 -> 220
- moved C6 5.66 mm to (188.5, 83.2), turned to 180 degrees
- moved J1 2.14 mm to (196.3, 69.7)
- moved GND1 1.25 mm to (126.0, 61.6)
- renumbered GND to GND1, GND to GND2, Vd to Vd1, Vf to Vf1, Vop to Vop1
Connections:
- J1 pad 5: /Vref -> /Vsel
- J1 pad 6: /Vsel -> /Vref
Routing:
- net /Vsel: track 45.0 -> 87.5 mm
- net /Vreg: track 129.0 -> 148.6 mm
- net /+VPOSA: track 63.0 -> 75.1 mm
- net /-VPOSA: track 41.8 -> 49.1 mm
- net /Vref: track 131.1 -> 132.6 mm
- net Net-(Q7-E): track 49.0 -> 50.4 mm
- net Net-(Q1-B): track 19.6 -> 20.5 mm
- net Net-(R17-Pad1): track 33.8 -> 34.4 mm
- net /Vo: track 24.5 -> 25.1 mm
Other:
- board size 74.8 x 50.7 mm -> 80.9 x 50.7 mm

Commit message: pcb_para_imprimir
Parts:
- added R24: 10, Resistor_THT:R_Axial_DIN0207_L6.3mm_D2.5mm_P7.62mm_Horizontal, F.Cu at (127.5, 84.3)
- added R25: 10, Resistor_THT:R_Axial_DIN0207_L6.3mm_D2.5mm_P7.62mm_Horizontal, F.Cu at (127.5, 81.3)
- moved Q4 7.62 mm to (129.6, 69.6)
- moved Q5 7.37 mm to (135.2, 69.7)
- moved Q2 6.30 mm to (129.5, 73.5)
- moved Q6 6.15 mm to (135.2, 73.6)
- moved RE2 6.07 mm to (132.7, 54.3)
- moved RE1 6.04 mm to (129.6, 54.3)
- moved Vd1 4.83 mm to (131.9, 50.8)
- moved GND1 4.34 mm to (124.1, 57.7)
- moved R1 3.75 mm to (124.7, 66.3)
- moved Rcp1 2.83 mm to (138.6, 55.9)
- moved C1 2.67 mm to (138.5, 66.5)
- moved Q7 1.63 mm to (136.6, 48.2)
- moved Q1 1.38 mm to (129.4, 86.9)
- moved Q3 1.38 mm to (134.3, 86.9)
- moved C3 1.03 mm to (140.9, 70.6)
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Connections:
- Q3 pad 1: Net-(Q2-E) -> Net-(Q3-C)
- Q6 pad 3: Net-(Q2-E) -> Net-(Q6-E)
Routing:
- net Net-(Q3-C): track 0.00 -> 11.9 mm
- net /Vlc: track 48.4 -> 37.6 mm
- net /Vreg: track 148.6 -> 153.8 mm
- net /Vf: track 53.6 -> 58.1 mm
- net Net-(Q1-B): track 20.5 -> 24.0 mm
- net Net-(Q6-E): track 0.00 -> 2.66 mm
- net /+VPOSA: track 75.1 -> 72.5 mm
- net Net-(Q5-E): track 6.00 -> 3.70 mm
- net Net-(Q4-E): track 4.43 -> 2.57 mm
- net Net-(Q2-C): track 10.4 -> 12.1 mm
- net Net-(Q7-E): track 50.4 -> 48.8 mm
- net Net-(R17-Pad1): track 34.4 -> 35.8 mm
- net Net-(Q2-E): track 7.64 -> 8.90 mm
- net /Vref: track 132.6 -> 131.5 mm
- net Net-(U1A-+): track 19.5 -> 18.8 mm
Other:
- board size 80.9 x 50.7 mm -> 83.3 x 51.5 mm
- board text added: "Vref Vsel Vreg +VP -VP GND"
- board text removed: "Vsel Vref Vreg +VP -VP GND"

Commit message: ojala no rompa todo
Parts:
- added C7: C, Capacitor_THT:CP_Radial_D5.0mm_P2.50mm, F.Cu at (160.6, 94.4)
- added R26: 1k, Resistor_THT:R_Axial_DIN0207_L6.3mm_D2.5mm_P7.62mm_Horizontal, F.Cu at (163.8, 94.4)
- added R27: 1k, Resistor_THT:R_Axial_DIN0207_L6.3mm_D2.5mm_P7.62mm_Horizontal, F.Cu at (163.8, 86.4)
- GND1, GND2, Vd1, Vf1, Vop1: footprint LDO_C2:TestPoint_THTPad_1.3x1.3mm_Drill0.7mm -> TestPoint:TestPoint_THTPad_2.0x2.0mm_Drill1.0mm
- J1: footprint LDO_C2:TerminalBlock_4Ucon_1x06_P3.50mm_Horizontal -> TerminalBlock:TerminalBlock_bornier-6_P5.08mm
- J2: footprint LDO_C2:TerminalBlock_4Ucon_1x02_P3.50mm_Horizontal(3D) -> TerminalBlock:TerminalBlock_bornier-2_P5.08mm
- Rs1: footprint Resistor_THT:R_Axial_DIN0207_L6.3mm_D2.5mm_P7.62mm_Horizontal -> Resistor_THT:R_Axial_Power_L25.0mm_W6.4mm_P30.48mm
- moved Rs1 23.5 mm to (183.4, 47.3)
- moved GND2 18.8 mm to (200.9, 47.3)
- moved J1 12.7 mm to (200.8, 57.8)
- moved J2 12.3 mm to (188.5, 47.3), turned to 0 degrees
- moved C9 8.67 mm to (188.2, 67.2), turned to -90 degrees
- moved C4 7.25 mm to (192.6, 61.4)
- moved C5 6.89 mm to (192.5, 67.9)
- moved Q8 5.63 mm to (142.5, 45.0)
- moved C2 4.55 mm to (190.6, 74.7)
- moved C6 4.21 mm to (190.6, 79.5)
- moved J3 3.35 mm to (189.1, 84.7)
- moved R3 3.28 mm to (167.8, 90.0)
- moved C10 3.01 mm to (188.2, 61.3), turned to -90 degrees
- moved R2 2.32 mm to (182.7, 63.6)
- moved R18 1.22 mm to (147.2, 79.2)
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Connections:
- M1 pad 2: /Vsel -> Net-(M1-G)
Routing:
- net /Vsel: track 87.5 -> 64.6 mm
- net Net-(M1-G): track 0.00 -> 21.6 mm
- net Net-(Q7-E): track 48.8 -> 60.2 mm
- net /-VPOSA: track 49.1 -> 42.9 mm
- net /+VPOSA: track 72.5 -> 68.0 mm
- net /Vref: track 131.5 -> 135.2 mm
- net Net-(R3-Pad1): track 3.19 -> 6.50 mm
- net Net-(R19-Pad2): track 8.19 -> 11.0 mm
- net Net-(Q7-C): track 10.3 -> 13.0 mm
- net Net-(R2-Pad1): track 3.50 -> 6.03 mm
- net /Vo: track 25.1 -> 27.5 mm
- net /Vf: track 58.1 -> 55.7 mm
- net /Sum: track 47.4 -> 46.2 mm
- net Net-(R17-Pad1): track 35.8 -> 36.9 mm
- net Net-(Q2-E): track 8.90 -> 9.97 mm
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Other:
- board size 83.3 x 51.5 mm -> 89.8 x 61.1 mm
- board text removed: "Circuito 3.3V/5V Grupo 5"
- board text removed: "LDO"
- board text removed: "Vref Vsel Vreg +VP -VP GND"

Commit message: nuevo pcb
Parts:
- moved GND2 19.6 mm to (183.2, 55.8)
- moved GND1 3.79 mm to (123.3, 54.0)
- moved R17 3.71 mm to (149.4, 62.4)
- moved Vf1 2.16 mm to (139.9, 80.1)
- moved Q9 2.03 mm to (143.8, 52.8)
- moved C6 2.03 mm to (192.6, 79.7)
- moved R13 1.96 mm to (143.4, 91.9)
- moved R12 1.96 mm to (140.1, 84.3)
- moved R14 1.96 mm to (146.9, 84.3)
- moved R3 1.57 mm to (169.4, 90.2)
- moved R8 1.50 mm to (176.8, 83.3)
- moved Rcp1 1.48 mm to (140.0, 55.6)
- moved RE1 1.46 mm to (128.1, 54.2)
- moved R15 1.37 mm to (150.4, 89.7)
- moved R23 1.17 mm to (169.2, 52.8)
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Connections:
- Q8 pad 1: Net-(Q7-E) -> Net-(Q7-C)
- Q8 pad 2: Net-(Q7-C) -> Net-(Q7-E)
Routing:
- net /Vf: track 55.7 -> 62.9 mm
- net Net-(Q7-C): track 13.0 -> 7.89 mm
- net /Vlc: track 38.2 -> 41.6 mm
- net Net-(M1-G): track 21.6 -> 24.2 mm
- net /Vref: track 135.2 -> 137.3 mm
- net /Vsel: track 64.6 -> 66.6 mm
- net Net-(R7-Pad2): track 3.97 -> 5.92 mm
- net Net-(R11-Pad2): track 5.36 -> 6.89 mm
- net /Vreg: track 153.3 -> 154.8 mm
- net Net-(U1B--): track 23.3 -> 24.4 mm
- net Net-(R14-Pad2): track 3.53 -> 4.45 mm
- net /Vo: track 27.5 -> 26.7 mm
- net Net-(R17-Pad1): track 36.9 -> 36.1 mm
- net Net-(R3-Pad1): track 6.50 -> 7.32 mm
- net Net-(Q9-E): track 2.77 -> 3.54 mm
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Other:
- board size 89.8 x 61.1 mm -> 89.2 x 62.1 mm
- board text added: "LDO 3.3V/5V Grupo 5"

Commit message: a
Parts:
- GND1, GND2, Vd1, Vf1, Vop1: footprint TestPoint:TestPoint_THTPad_2.0x2.0mm_Drill1.0mm -> LDO_C2:TestPoint_THTPad_2.0x2.0mm_Drill1.0mm
- J1: footprint TerminalBlock:TerminalBlock_bornier-6_P5.08mm -> LDO_C2:TerminalBlock_bornier-6_P5.08mm
- J2: footprint TerminalBlock:TerminalBlock_bornier-2_P5.08mm -> LDO_C2:TerminalBlock_bornier-2_P5.08mm
Other:
- board text added: "Vo GND"
- board text added: "Vref Vsel Vreg +VP -VP GND"
- board text removed: "GND Vo"
Changed lines of the file:
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@@
 		)
 	)
-	(footprint "TestPoint:TestPoint_THTPad_2.0x2.0mm_Drill1.0mm"
+	(footprint "LDO_C2:TestPoint_THTPad_2.0x2.0mm_Drill1.0mm"
 		(layer "F.Cu")
 		(at 148.6 67.6)
@@
 		(tags "test point THT pad rectangle square")
 		(property "Reference" "Vop1"
-			(at 0.1 -2.8 0)
+			(at 0.1 2.5 0)
 			(layer "F.SilkS")
 			(effects
@@
 			)
 		)
-		(property "Footprint" "TestPoint:TestPoint_THTPad_2.0x2.0mm_Drill1.0mm"
+		(property "Footprint" "LDO_C2:TestPoint_THTPad_2.0x2.0mm_Drill1.0mm"
 			(at 0 0 0)
 			(unlocked yes)
@@
 			(pintype "passive")
 		)
+		(model "${KIPRJMOD}/Modelos3D/male_pin.wrl"
+			(offset
+				(xyz -19.35 0 0)
+			)
+			(scale
+				(xyz 0.3 0.3 0.3)
+			)
+			(rotate
+				(xyz -90 0 0)
+			)
+		)
 	)
 	(footprint "Package_TO_SOT_THT:TO-92L_Inline_Wide"
@@
 		)
 	)
-	(footprint "TestPoint:TestPoint_THTPad_2.0x2.0mm_Drill1.0mm"
+	(footprint "LDO_C2:TestPoint_THTPad_2.0x2.0mm_Drill1.0mm"
 		(layer "F.Cu")
 		(at 139.9 80.1)
@@
 		(tags "test point THT pad rectangle square")
 		(property "Reference" "Vf1"
-			(at 0 -2.4 0)
+			(at 0.1 2.5 0)
 			(layer "F.SilkS")
 			(effects
@@
 			)
 		)
-		(property "Footprint" "TestPoint:TestPoint_THTPad_2.0x2.0mm_Drill1.0mm"
+		(property "Footprint" "LDO_C2:TestPoint_THTPad_2.0x2.0mm_Drill1.0mm"
 			(at 0 0 0)
 			(unlocked yes)
@@
 			(pintype "passive")
 		)
+		(model "${KIPRJMOD}/Modelos3D/male_pin.wrl"
+			(offset
+				(xyz -19.35 0 0)
+			)
+			(scale
+				(xyz 0.3 0.3 0.3)
+			)
+			(rotate
+				(xyz -90 0 0)
+			)
+		)
 	)
 	(footprint "Resistor_THT:R_Axial_DIN0207_L6.3mm_D2.5mm_P7.62mm_Horizontal"
@@
 		)
 	)
-	(footprint "TestPoint:TestPoint_THTPad_2.0x2.0mm_Drill1.0mm"
+	(footprint "LDO_C2:TestPoint_THTPad_2.0x2.0mm_Drill1.0mm"
 		(layer "F.Cu")
 		(at 131.9 50.825)
@@
 		(tags "test point THT pad rectangle square")
 		(property "Reference" "Vd1"
-			(at 0 -1.998 0)
+			(at 0.1 2.5 0)
 			(layer "F.SilkS")
 			(effects
@@
 			)
 		)
-		(property "Footprint" "TestPoint:TestPoint_THTPad_2.0x2.0mm_Drill1.0mm"
+		(property "Footprint" "LDO_C2:TestPoint_THTPad_2.0x2.0mm_Drill1.0mm"
 			(at 0 0 0)
 			(unlocked yes)
@@
 			(pintype "passive")
 		)
+		(model "${KIPRJMOD}/Modelos3D/male_pin.wrl"
+			(offset
+				(xyz -19.35 0 0)
+			)
+			(scale
+				(xyz 0.3 0.3 0.3)
+			)
+			(rotate
+				(xyz -90 0 0)
+			)
+		)
 	)
 	(footprint "Resistor_THT:R_Axial_DIN0207_L6.3mm_D2.5mm_P7.62mm_Horizontal"
@@
 		)
 	)
-	(footprint "TestPoint:TestPoint_THTPad_2.0x2.0mm_Drill1.0mm"
+	(footprint "LDO_C2:TestPoint_THTPad_2.0x2.0mm_Drill1.0mm"
 		(layer "F.Cu")
 		(at 183.2 55.8)
@@
 		(tags "test point THT pad rectangle square")
 		(property "Reference" "GND2"
-			(at 0.1 -2.9 0)
+			(at 0.1 2.5 0)
 			(layer "F.SilkS")
 			(effects
@@
 			)
 		)
-		(property "Footprint" "TestPoint:TestPoint_THTPad_2.0x2.0mm_Drill1.0mm"
+		(property "Footprint" "LDO_C2:TestPoint_THTPad_2.0x2.0mm_Drill1.0mm"
 			(at 0 0 0)
 			(unlocked yes)
@@
 			(pintype "passive")
 		)
+		(model "${KIPRJMOD}/Modelos3D/male_pin.wrl"
+			(offset
+				(xyz -19.35 0 0)
+			)
+			(scale
+				(xyz 0.3 0.3 0.3)
+			)
+			(rotate
+				(xyz -90 0 0)
+			)
+		)
 	)
 	(footprint "Capacitor_THT:CP_Radial_D5.0mm_P2.50mm"
@@
 		(tags "Resistor Axial_DIN0207 series Axial Horizontal pin pitch 7.62mm 0.25W = 1/4W length 6.3mm diameter 2.5mm")
 		(property "Reference" "R5"
-			(at -1.83 -0.03 180)
+			(at 3.77 -0.03 -90)
 			(layer "F.SilkS")
 			(effects
@@
 		(tags "Resistor Axial_DIN0207 series Axial Horizontal pin pitch 7.62mm 0.25W = 1/4W length 6.3mm diameter 2.5mm")
 		(property "Reference" "R2"
-			(at 9.4 0.08 180)
+			(at 3.785 0.05 -90)
 			(layer "F.SilkS")
 			(effects
@@
 		)
 	)
-	(footprint "TerminalBlock:TerminalBlock_bornier-2_P5.08mm"
+	(footprint "LDO_C2:TerminalBlock_bornier-2_P5.08mm"
 		(layer "F.Cu")
 		(at 188.5 47.325)
@@
 		(tags "terminal block bornier2")
 		(property "Reference" "J2"
-			(at 2.54 -5.08 0)
+			(at 2.7 -2.525 0)
 			(layer "F.SilkS")
 			(effects
@@
 			)
 		)
-		(property "Footprint" "TerminalBlock:TerminalBlock_bornier-2_P5.08mm"
+		(property "Footprint" "LDO_C2:TerminalBlock_bornier-2_P5.08mm"
 			(at 0 0 0)
 			(unlocked yes)
@@
 			(pintype "passive")
 		)
-		(model "${KICAD8_3DMODEL_DIR}/TerminalBlock.3dshapes/TerminalBlock_bornier-2_P5.08mm.wrl"
+		(model "${KIPRJMOD}/Modelos3D/Bornerax2.wrl"
 			(offset
-				(xyz 2.539999962 0 0)
+				(xyz 132.5 -41.5 -16)
 			)
 			(scale
-				(xyz 1 1 1)
+				(xyz 0.4 0.4 0.4)
 			)
 			(rotate
-				(xyz 0 0 0)
+				(xyz 0 0 -90)
 			)
 		)
@@
 		)
 	)
-	(footprint "TestPoint:TestPoint_THTPad_2.0x2.0mm_Drill1.0mm"
+	(footprint "LDO_C2:TestPoint_THTPad_2.0x2.0mm_Drill1.0mm"
 		(layer "F.Cu")
 		(at 123.3 54)
@@
 			)
 		)
-		(property "Footprint" "TestPoint:TestPoint_THTPad_2.0x2.0mm_Drill1.0mm"
+		(property "Footprint" "LDO_C2:TestPoint_THTPad_2.0x2.0mm_Drill1.0mm"
 			(at 0 0 0)
 			(unlocked yes)
@@
 			(pintype "passive")
 		)
+		(model "${KIPRJMOD}/Modelos3D/male_pin.wrl"
+			(offset
+				(xyz -19.35 0 0)
+			)
+			(scale
+				(xyz 0.3 0.3 0.3)
+			)
+			(rotate
+				(xyz -90 0 0)
+			)
+		)
 	)
-	(footprint "TerminalBlock:TerminalBlock_bornier-6_P5.08mm"
+	(footprint "LDO_C2:TerminalBlock_bornier-6_P5.08mm"
 		(layer "F.Cu")
 		(at 200.825 57.8 -90)
@@
 		(tags "terminal block bornier6")
 		(property "Reference" "J1"
-			(at 12.65 -4.55 -90)
+			(at 12.65 -5.375 90)
 			(layer "F.SilkS")
 			(effects
@@
 		)
 		(property "Value" "Conn_01x06_Socket"
-			(at 12.7 4.75 -90)
+			(at 12.7 4.75 90)
 			(layer "F.Fab")
 			(effects
@@
 			)
 		)
-		(property "Footprint" "TerminalBlock:TerminalBlock_bornier-6_P5.08mm"
+		(property "Footprint" "LDO_C2:TerminalBlock_bornier-6_P5.08mm"
 			(at 0 0 -90)
 			(unlocked yes)
@@
 		)
 		(fp_text user "${REFERENCE}"
-			(at 12.7 0 -90)
+			(at 12.7 0 90)
 			(layer "F.Fab")
 			(effects
@@
 			(pintype "passive")
 		)
-		(model "${KICAD8_3DMODEL_DIR}/TerminalBlock.3dshapes/TerminalBlock_bornier-6_P5.08mm.wrl"
+		(model "${KIPRJMOD}/Modelos3D/Bornerax2.wrl"
 			(offset
-				(xyz 12.69999981 0 0)
+				(xyz 132.5 -41.59 -16)
 			)
 			(scale
-				(xyz 1 1 1)
+				(xyz 0.4 0.4 0.4)
 			)
 			(rotate
-				(xyz 0 0 0)
+				(xyz 0 0 -90)
+			)
+		)
+		(model "${KIPRJMOD}/Modelos3D/Bornerax2.wrl"
+			(offset
+				(xyz 142.7 -41.59 -16)
+			)
+			(scale
+				(xyz 0.4 0.4 0.4)
+			)
+			(rotate
+				(xyz 0 0 -90)
+			)
+		)
+		(model "${KIPRJMOD}/Modelos3D/Bornerax2.wrl"
+			(offset
+				(xyz 152.9 -41.59 -16)
+			)
+			(scale
+				(xyz 0.4 0.4 0.4)
+			)
+			(rotate
+				(xyz 0 0 -90)
 			)
 		)
@@
 	)
 	(gr_text "Circuito LDO 3.3V/5V\nGrupo 5"
-		(at 178.9 57.1 0)
+		(at 132.9 98.7 0)
 		(layer "F.SilkS")
 		(effects
@@
 		)
 	)
-	(gr_text "GND   Vo"
-		(at 194 52 180)
+	(gr_text "Vo    GND"
+		(at 188.2 51.1 0)
+		(layer "F.SilkS")
+		(effects
+			(font
+				(size 0.8 0.8)
+				(thickness 0.15)
+				(bold yes)
+			)
+			(justify left bottom)
+		)
+	)
+	(gr_text "Vref     Vsel    Vreg    +VP    -VP    GND"
+		(at 204.1 84.7 90)
 		(layer "F.SilkS")
 		(effects
