File: Checkpoint 2/DCE - PCB - v1/dce-pcb-v1.kicad_sch (KiCad schematic)
At the start: 55 parts, among them J2 Conn_01x02_Socket

Commit message: avance pcb
Parts:
- C4, C5, C6, C7, C8: footprint Capacitor_THT:C_Disc_D3.4mm_W2.1mm_P2.50mm -> Capacitor_THT:CP_Radial_D5.0mm_P2.00mm
Changed lines of the file:
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@@
 			)
 		)
-		(property "Footprint" "Capacitor_THT:C_Disc_D3.4mm_W2.1mm_P2.50mm"
+		(property "Footprint" "Capacitor_THT:CP_Radial_D5.0mm_P2.00mm"
 			(at 265.43 170.4848 0)
 			(effects
@@
 			)
 		)
-		(property "Footprint" "Capacitor_THT:C_Disc_D3.4mm_W2.1mm_P2.50mm"
+		(property "Footprint" "Capacitor_THT:CP_Radial_D5.0mm_P2.00mm"
 			(at 265.43 179.3748 0)
 			(effects
@@
 			)
 		)
-		(property "Footprint" "Capacitor_THT:C_Disc_D3.4mm_W2.1mm_P2.50mm"
+		(property "Footprint" "Capacitor_THT:CP_Radial_D5.0mm_P2.00mm"
 			(at 265.43 160.3248 0)
 			(effects
@@
 			)
 		)
-		(property "Footprint" "Capacitor_THT:C_Disc_D3.4mm_W2.1mm_P2.50mm"
+		(property "Footprint" "Capacitor_THT:CP_Radial_D5.0mm_P2.00mm"
 			(at 265.43 152.7048 0)
 			(effects
@@
 			)
 		)
-		(property "Footprint" "Capacitor_THT:C_Disc_D3.4mm_W2.1mm_P2.50mm"
+		(property "Footprint" "Capacitor_THT:CP_Radial_D5.0mm_P2.00mm"
 			(at 265.43 143.8148 0)
 			(effects

Commit message: Actualizacion PCB
Connections:
- net Vref: now also C7.1, J?.5 (Pin_5); no longer C6.1, J?.4 (Pin_4)
- net Vreg: now also C6.1, J?.4 (Pin_4); no longer C7.1, J?.5 (Pin_5)
Changed lines of the file:
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@@
 		)
 	)
-	(label "Vref"
+	(label "Vreg"
 		(at 251.46 161.29 90)
 		(fields_autoplaced yes)
@@
 		)
 	)
-	(label "Vreg"
+	(label "Vref"
 		(at 248.92 153.67 90)
 		(fields_autoplaced yes)

Commit message: PCB actualizado
Parts:
- added TP5: TestPoint, TestPoint:TestPoint_THTPad_1.0x1.0mm_Drill0.5mm, symbol Connector:TestPoint
- C4, C5, C6, C7, C8: footprint Capacitor_THT:CP_Radial_D5.0mm_P2.00mm -> Capacitor_THT:CP_Radial_D5.0mm_P2.50mm
- M?, Q? (x8): footprint Package_TO_SOT_THT:TO-92L_Inline -> Package_TO_SOT_THT:TO-92L_Inline_Wide
Connections:
- net 0: now also TP5.1
Changed lines of the file:
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@@
 			)
 		)
-		(property "Footprint" "Capacitor_THT:CP_Radial_D5.0mm_P2.00mm"
+		(property "Footprint" "Capacitor_THT:CP_Radial_D5.0mm_P2.50mm"
 			(at 265.43 170.4848 0)
 			(effects
@@
 			)
 		)
-		(property "Footprint" "Package_TO_SOT_THT:TO-92L_Inline"
+		(property "Footprint" "Package_TO_SOT_THT:TO-92L_Inline_Wide"
 			(at 142.24 38.1 0)
 			(effects
@@
 			)
 		)
-		(property "Footprint" "Capacitor_THT:CP_Radial_D5.0mm_P2.00mm"
+		(property "Footprint" "Capacitor_THT:CP_Radial_D5.0mm_P2.50mm"
 			(at 265.43 179.3748 0)
 			(effects
@@
 			)
 		)
-		(property "Footprint" "Package_TO_SOT_THT:TO-92L_Inline"
+		(property "Footprint" "Package_TO_SOT_THT:TO-92L_Inline_Wide"
 			(at 121.92 130.81 0)
 			(effects
@@
 			)
 		)
-		(property "Footprint" "Package_TO_SOT_THT:TO-92L_Inline"
+		(property "Footprint" "Package_TO_SOT_THT:TO-92L_Inline_Wide"
 			(at 92.71 67.31 0)
 			(effects
@@
 			)
 		)
-		(property "Footprint" "Package_TO_SOT_THT:TO-92L_Inline"
+		(property "Footprint" "Package_TO_SOT_THT:TO-92L_Inline_Wide"
 			(at 185.42 85.09 0)
 			(effects
@@
 	)
 	(symbol
+		(lib_id "Connector:TestPoint")
+		(at 78.74 102.87 270)
+		(unit 1)
+		(exclude_from_sim no)
+		(in_bom yes)
+		(on_board yes)
+		(dnp no)
+		(property "Reference" "TP5"
+			(at 84.328 106.172 90)
+			(effects
+				(font
+					(size 1.27 1.27)
+				)
+			)
+		)
+		(property "Value" "TestPoint"
+			(at 84.582 104.648 90)
+			(effects
+				(font
+					(size 1.27 1.27)
+				)
+			)
+		)
+		(property "Footprint" "TestPoint:TestPoint_THTPad_1.0x1.0mm_Drill0.5mm"
+			(at 78.74 107.95 0)
+			(effects
+				(font
+					(size 1.27 1.27)
+				)
+				(hide yes)
+			)
+		)
+		(property "Datasheet" "~"
+			(at 78.74 107.95 0)
+			(effects
+				(font
+					(size 1.27 1.27)
+				)
+				(hide yes)
+			)
+		)
+		(property "Description" "test point"
+			(at 78.74 102.87 0)
+			(effects
+				(font
+					(size 1.27 1.27)
+				)
+				(hide yes)
+			)
+		)
+		(pin "1"
+		)
+		(instances
+			(project "dce-pcb-v1"
+				(path "/e6ededfa-1272-42e1-ab55-13acb1f29d6e"
+					(reference "TP5")
+					(unit 1)
+				)
+			)
+		)
+	)
+	(symbol
 		(lib_id "ltspice:npn")
 		(at 73.66 88.9 0)
@@
 			)
 		)
-		(property "Footprint" "Package_TO_SOT_THT:TO-92L_Inline"
+		(property "Footprint" "Package_TO_SOT_THT:TO-92L_Inline_Wide"
 			(at 73.66 88.9 0)
 			(effects
@@
 			)
 		)
-		(property "Footprint" "Package_TO_SOT_THT:TO-92L_Inline"
+		(property "Footprint" "Package_TO_SOT_THT:TO-92L_Inline_Wide"
 			(at 64.77 67.31 0)
 			(effects
@@
 			)
 		)
-		(property "Footprint" "Package_TO_SOT_THT:TO-92L_Inline"
+		(property "Footprint" "Package_TO_SOT_THT:TO-92L_Inline_Wide"
 			(at 82.55 55.88 0)
 			(effects
@@
 			)
 		)
-		(property "Footprint" "Capacitor_THT:CP_Radial_D5.0mm_P2.00mm"
+		(property "Footprint" "Capacitor_THT:CP_Radial_D5.0mm_P2.50mm"
 			(at 265.43 160.3248 0)
 			(effects
@@
 			)
 		)
-		(property "Footprint" "Package_TO_SOT_THT:TO-92L_Inline"
+		(property "Footprint" "Package_TO_SOT_THT:TO-92L_Inline_Wide"
 			(at 74.93 55.88 0)
 			(effects
@@
 			)
 		)
-		(property "Footprint" "Package_TO_SOT_THT:TO-92L_Inline"
+		(property "Footprint" "Package_TO_SOT_THT:TO-92L_Inline_Wide"
 			(at 35.56 88.9 0)
 			(effects
@@
 			)
 		)
-		(property "Footprint" "Capacitor_THT:CP_Radial_D5.0mm_P2.00mm"
+		(property "Footprint" "Capacitor_THT:CP_Radial_D5.0mm_P2.50mm"
 			(at 265.43 152.7048 0)
 			(effects
@@
 			)
 		)
-		(property "Footprint" "Capacitor_THT:CP_Radial_D5.0mm_P2.00mm"
+		(property "Footprint" "Capacitor_THT:CP_Radial_D5.0mm_P2.50mm"
 			(at 265.43 143.8148 0)
 			(effects

Commit message: actualizacion PCB
Parts:
- GND1: renamed from TP5; footprint TestPoint:TestPoint_THTPad_1.0x1.0mm_Drill0.5mm -> LDO_C2:TestPoint_THTPad_1.3x1.3mm_Drill0.7mm
- GND2: renamed from TP4; footprint TestPoint:TestPoint_THTPad_1.0x1.0mm_Drill0.5mm -> LDO_C2:TestPoint_THTPad_1.3x1.3mm_Drill0.7mm
- J2: footprint TerminalBlock_4Ucon:TerminalBlock_4Ucon_1x02_P3.50mm_Horizontal -> LDO_C2:TerminalBlock_4Ucon_1x02_P3.50mm_Horizontal(3D)
- J?: footprint TerminalBlock_4Ucon:TerminalBlock_4Ucon_1x06_P3.50mm_Horizontal -> LDO_C2:TerminalBlock_4Ucon_1x06_P3.50mm_Horizontal
- U? (x5): footprint Package_DIP:DIP-14_W7.62mm_Socket -> LDO_C2:DIP-14_W7.62mm_Socket
- Vd1: renamed from TP2; footprint TestPoint:TestPoint_THTPad_1.0x1.0mm_Drill0.5mm -> LDO_C2:TestPoint_THTPad_1.3x1.3mm_Drill0.7mm
- Vf1: renamed from TP1; footprint TestPoint:TestPoint_THTPad_1.0x1.0mm_Drill0.5mm -> LDO_C2:TestPoint_THTPad_1.3x1.3mm_Drill0.7mm
- Vop1: renamed from TP3; footprint TestPoint:TestPoint_THTPad_1.0x1.0mm_Drill0.5mm -> LDO_C2:TestPoint_THTPad_1.3x1.3mm_Drill0.7mm
Changed lines of the file:
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@@
 	(paper "A4")
 	(junction
+		(at 135.89 134.62)
+		(diameter 0)
+		(color 0 0 0 0)
+	)
+	(junction
 		(at 269.24 180.34)
 		(diameter 0)
@@
 	)
 	(junction
-		(at 110.49 57.15)
+		(at 160.02 49.53)
 		(diameter 0)
 		(color 0 0 0 0)
 	)
 	(junction
-		(at 160.02 49.53)
+		(at 240.03 49.53)
 		(diameter 0)
 		(color 0 0 0 0)
 	)
 	(junction
-		(at 240.03 49.53)
+		(at 266.7 58.42)
 		(diameter 0)
 		(color 0 0 0 0)
@@
 	)
 	(junction
-		(at 123.19 71.12)
-		(diameter 0)
-		(color 0 0 0 0)
-	)
-	(junction
-		(at 266.7 58.42)
-		(diameter 0)
-		(color 0 0 0 0)
-	)
-	(junction
 		(at 30.48 85.09)
 		(diameter 0)
@@
 	)
 	(junction
-		(at 135.89 134.62)
+		(at 123.19 71.12)
 		(diameter 0)
 		(color 0 0 0 0)
@@
 	)
 	(junction
+		(at 110.49 57.15)
+		(diameter 0)
+		(color 0 0 0 0)
+	)
+	(junction
 		(at 52.07 144.78)
 		(diameter 0)
@@
 	(wire
 		(pts
-			(xy 110.49 57.15) (xy 118.11 57.15)
-		)
-		(stroke
-			(width 0)
-			(type default)
-		)
-	)
-	(wire
-		(pts
 			(xy 233.68 91.44) (xy 233.68 85.09)
 		)
@@
 	(wire
 		(pts
-			(xy 266.7 58.42) (xy 266.7 60.96)
+			(xy 266.7 52.07) (xy 266.7 58.42)
 		)
 		(stroke
@@
 	(wire
 		(pts
-			(xy 139.7 134.62) (xy 135.89 134.62)
-		)
-		(stroke
-			(width 0.1524)
-			(type solid)
-		)
-	)
-	(wire
-		(pts
 			(xy 146.05 58.42) (xy 146.05 71.12)
 		)
@@
 	(wire
 		(pts
-			(xy 266.7 52.07) (xy 266.7 58.42)
-		)
-		(stroke
-			(width 0)
-			(type default)
-		)
-	)
-	(wire
-		(pts
 			(xy 91.44 57.15) (xy 110.49 57.15)
 		)
@@
 	(wire
 		(pts
-			(xy 135.89 134.62) (xy 130.81 134.62)
+			(xy 130.81 134.62) (xy 135.89 134.62)
 		)
 		(stroke
@@
 	(wire
 		(pts
-			(xy 101.6 71.12) (xy 123.19 71.12)
-		)
-		(stroke
-			(width 0.1524)
-			(type solid)
-		)
-	)
-	(wire
-		(pts
 			(xy 139.7 134.62) (xy 139.7 149.86)
 		)
@@
 	(wire
 		(pts
+			(xy 123.19 71.12) (xy 146.05 71.12)
+		)
+		(stroke
+			(width 0.1524)
+			(type solid)
+		)
+	)
+	(wire
+		(pts
 			(xy 95.25 146.05) (xy 88.9 146.05)
 		)
@@
 	(wire
 		(pts
+			(xy 135.89 134.62) (xy 139.7 134.62)
+		)
+		(stroke
+			(width 0.1524)
+			(type solid)
+		)
+	)
+	(wire
+		(pts
 			(xy 265.43 153.67) (xy 269.24 153.67)
 		)
@@
 	(wire
 		(pts
-			(xy 123.19 71.12) (xy 146.05 71.12)
+			(xy 101.6 71.12) (xy 123.19 71.12)
 		)
 		(stroke
@@
 	(wire
 		(pts
+			(xy 110.49 57.15) (xy 118.11 57.15)
+		)
+		(stroke
+			(width 0)
+			(type default)
+		)
+	)
+	(wire
+		(pts
 			(xy 69.85 31.75) (xy 69.85 26.67)
 		)
@@
 	(wire
 		(pts
+			(xy 266.7 58.42) (xy 266.7 60.96)
+		)
+		(stroke
+			(width 0)
+			(type default)
+		)
+	)
+	(wire
+		(pts
 			(xy 30.48 88.9) (xy 30.48 85.09)
 		)
@@
 			)
 		)
-		(property "Footprint" "TerminalBlock_4Ucon:TerminalBlock_4Ucon_1x02_P3.50mm_Horizontal"
+		(property "Footprint" "LDO_C2:TerminalBlock_4Ucon_1x02_P3.50mm_Horizontal(3D)"
 			(at 271.78 49.53 0)
 			(effects
@@
 		(on_board yes)
 		(dnp no)
-		(property "Reference" "TP3"
+		(property "Reference" "Vop1"
 			(at 134.112 125.984 0)
 			(effects
@@
 			)
 		)
-		(property "Footprint" "TestPoint:TestPoint_THTPad_1.0x1.0mm_Drill0.5mm"
+		(property "Footprint" "LDO_C2:TestPoint_THTPad_1.3x1.3mm_Drill0.7mm"
 			(at 140.97 134.62 0)
 			(effects
@@
 			(project "dce-pcb-v1"
 				(path "/e6ededfa-1272-42e1-ab55-13acb1f29d6e"
-					(reference "TP3")
+					(reference "Vop1")
 					(unit 1)
 				)
@@
 		(on_board yes)
 		(dnp no)
-		(property "Reference" "TP2"
+		(property "Reference" "Vd1"
 			(at 108.458 48.006 0)
 			(effects
@@
 			)
 		)
-		(property "Footprint" "TestPoint:TestPoint_THTPad_1.0x1.0mm_Drill0.5mm"
+		(property "Footprint" "LDO_C2:TestPoint_THTPad_1.3x1.3mm_Drill0.7mm"
 			(at 115.57 57.15 0)
 			(effects
@@
 			(project "dce-pcb-v1"
 				(path "/e6ededfa-1272-42e1-ab55-13acb1f29d6e"
-					(reference "TP2")
+					(reference "Vd1")
 					(unit 1)
 				)
@@
 		(on_board yes)
 		(dnp no)
-		(property "Reference" "TP4"
+		(property "Reference" "GND2"
 			(at 261.112 55.118 90)
 			(effects
@@
 			)
 		)
-		(property "Footprint" "TestPoint:TestPoint_THTPad_1.0x1.0mm_Drill0.5mm"
+		(property "Footprint" "LDO_C2:TestPoint_THTPad_1.3x1.3mm_Drill0.7mm"
 			(at 266.7 53.34 0)
 			(effects
@@
 			(project ""
 				(path "/e6ededfa-1272-42e1-ab55-13acb1f29d6e"
-					(reference "TP4")
+					(reference "GND2")
 					(unit 1)
 				)
@@
 		(on_board yes)
 		(dnp no)
-		(property "Reference" "TP5"
+		(property "Reference" "GND1"
 			(at 84.328 106.172 90)
 			(effects
@@
 			)
 		)
-		(property "Footprint" "TestPoint:TestPoint_THTPad_1.0x1.0mm_Drill0.5mm"
+		(property "Footprint" "LDO_C2:TestPoint_THTPad_1.3x1.3mm_Drill0.7mm"
 			(at 78.74 107.95 0)
 			(effects
@@
 			(project "dce-pcb-v1"
 				(path "/e6ededfa-1272-42e1-ab55-13acb1f29d6e"
-					(reference "TP5")
+					(reference "GND1")
 					(unit 1)
 				)
@@
 			)
 		)
-		(property "Footprint" "Package_DIP:DIP-14_W7.62mm_Socket"
+		(property "Footprint" "LDO_C2:DIP-14_W7.62mm_Socket"
 			(at 238.76 97.79 0)
 			(effects
@@
 			)
 		)
-		(property "Footprint" "TerminalBlock_4Ucon:TerminalBlock_4Ucon_1x06_P3.50mm_Horizontal"
+		(property "Footprint" "LDO_C2:TerminalBlock_4Ucon_1x06_P3.50mm_Horizontal"
 			(at 254 194.31 0)
 			(effects
@@
 			)
 		)
-		(property "Footprint" "Package_DIP:DIP-14_W7.62mm_Socket"
+		(property "Footprint" "LDO_C2:DIP-14_W7.62mm_Socket"
 			(at 68.58 116.84 0)
 			(effects
@@
 			)
 		)
-		(property "Footprint" "Package_DIP:DIP-14_W7.62mm_Socket"
+		(property "Footprint" "LDO_C2:DIP-14_W7.62mm_Socket"
 			(at 68.58 144.78 0)
 			(effects
@@
 		(dnp no)
 		(fields_autoplaced yes)
-		(property "Reference" "TP1"
+		(property "Reference" "Vf1"
 			(at 125.73 66.5479 0)
 			(effects
@@
 			)
 		)
-		(property "Footprint" "TestPoint:TestPoint_THTPad_1.0x1.0mm_Drill0.5mm"
+		(property "Footprint" "LDO_C2:TestPoint_THTPad_1.3x1.3mm_Drill0.7mm"
 			(at 128.27 71.12 0)
 			(effects
@@
 			(project ""
 				(path "/e6ededfa-1272-42e1-ab55-13acb1f29d6e"
-					(reference "TP1")
+					(reference "Vf1")
 					(unit 1)
 				)
@@
 			)
 		)
-		(property "Footprint" "Package_DIP:DIP-14_W7.62mm_Socket"
+		(property "Footprint" "LDO_C2:DIP-14_W7.62mm_Socket"
 			(at 148.59 132.08 0)
 			(effects
@@
 			)
 		)
-		(property "Footprint" "Package_DIP:DIP-14_W7.62mm_Socket"
+		(property "Footprint" "LDO_C2:DIP-14_W7.62mm_Socket"
 			(at 186.69 134.62 0)
 			(effects
