File: Checkpoint 2/DCE - PCB - v1/dce-pcb-v1.kicad_sch (KiCad schematic)
At the start: 56 parts, among them J2 Conn_01x02_Socket

Commit message: valor de resistencia de compensacion corregida en el esquematico
Parts:
- Rcp1: value 470 -> 220
Changed lines of the file:
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@@
 			)
 		)
-		(property "Value" "470"
+		(property "Value" "220"
 			(at 96.2152 60.6298 0)
 			(effects
