File: Checkpoint 4/pcb_buck/pcb_pwm/pcb_pwm.kicad_sch (KiCad schematic)
At the start: 20 parts, among them J1 Conn_01x04_Socket, J2 Conn_01x03_Socket, U1 TL082, U3 LM393

Commit message: pwm
Parts:
- removed R1: 89k, Resistor_THT:R_Axial_DIN0207_L6.3mm_D2.5mm_P7.62mm_Horizontal, symbol ltspice:res
- removed R2: 100k, Resistor_THT:R_Axial_DIN0207_L6.3mm_D2.5mm_P7.62mm_Horizontal, symbol ltspice:res
- added R8: 1k, Resistor_THT:R_Axial_DIN0207_L6.3mm_D2.5mm_P7.62mm_Horizontal, symbol ltspice:res
- added R9: 649, Resistor_THT:R_Axial_DIN0207_L6.3mm_D2.5mm_P7.62mm_Horizontal, symbol ltspice:res
- TP5: value Vref -> Verr
Connections:
- net 0: now also U1.5 (+), U3.2 (-), R9.2
- net Vo: no longer J1.4 (Pin_4)
- net Vsin: now also R8.2; no longer J2.1 (Pin_1)
- net at TP5.1, U3.5 (+): now also U1.1; no longer J2.2 (Pin_2)
- net at U1.3 (+): now also J2.2 (Pin_2), TP4.1
- new net: J2.1 (Pin_1), R8.1, R9.1
- new net Vref: J1.4 (Pin_4), U1.2 (-)
Other:
- moved on the sheet: U1A, U1C, U3C

Commit message: pcb pwm
Parts:
- removed J1: Conn_01x04_Socket, TerminalBlock:TerminalBlock_bornier-4_P5.08mm, symbol Connector:Conn_01x04_Socket
- removed R7: 2,7k, Resistor_THT:R_Axial_DIN0207_L6.3mm_D2.5mm_P7.62mm_Horizontal, symbol ltspice:res
- removed U3: LM393, Package_DIP:DIP-8_W7.62mm_Socket, symbol Comparator:LM393
- added C4: 10n, Capacitor_THT:C_Disc_D3.4mm_W2.1mm_P2.50mm, symbol Device:C
- added C5: 10u, Capacitor_THT:CP_Radial_D5.0mm_P2.50mm, symbol Device:C
- added D1: D_Schottky, Diode_THT:D_DO-27_P12.70mm_Horizontal, symbol Device:D_Schottky
- added J3: Conn_01x06_Socket, TerminalBlock:TerminalBlock_bornier-6_P5.08mm, symbol Connector:Conn_01x06_Socket
- added R1, R2: 10k, Resistor_THT:R_Axial_DIN0207_L6.3mm_D2.5mm_P7.62mm_Horizontal, symbol ltspice:res
- added R10, R11, R12, R13: 100k, Resistor_THT:R_Axial_DIN0207_L6.3mm_D2.5mm_P7.62mm_Horizontal, symbol ltspice:res
- added R14: 10, Resistor_THT:R_Axial_DIN0207_L6.3mm_D2.5mm_P7.62mm_Horizontal, symbol ltspice:res
- added U2: LM2901, Package_DIP:DIP-14_W7.62mm_Socket, symbol Comparator:LM2901
- R3: value 100k -> 220k
- R4: value 27k -> 5,1k
- R5: value 33k -> 39k
- R6: value 5,1k -> 8,2k
- R8: value 1k -> 120
- R9: value 649 -> 68
Connections:
- net 0: now also RV1.2, C4.2, C5.2, D1.2 (A), J3.1 (Pin_1), R12.2, R14.2, U2.11 (+), U2.5 (+), U2.9 (+); no longer R9.2, U1.4 (V-)
- net Vcc: now also J3.2 (Pin_2), R1.2, R2.2, U2.3 (V+)
- net Vo: now also D1.1 (K), J3.6 (Pin_6), R2.1, U2.1
- net Vref: now also J3.5 (Pin_5), R10.2; no longer U1.2 (-)
- net Vsin: now also J3.4 (Pin_4)
- net Verr: now reaches TP5.1, U1.1
- net Verr: now also R11.1, U2.6 (-)
- net Vtriang: now reaches C1.1, R4.1, TP3.1, U1.7
- net Vtriang: now also U2.7 (+)
- net at R3.2, R4.2: now also U2.4 (-)
- net Vcomp: now reaches J2.2 (Pin_2), TP4.1
- net Vcomp: now also R13.2; no longer U1.3 (+)
- net Vcuad: now reaches R3.1, R5.2, TP2.1
- net Vcuad: now also R1.1, U2.2
- new net: R10.1, R11.2, U1.2 (-)
- new net: R12.1, R13.1, U1.3 (+)
- new net: R14.1, R9.2
- new net: U2.14, U2.8 (-)
- new net: U2.10 (-), U2.13
- new net -Vcc: C4.1, C5.1, J3.3 (Pin_3), U1.4 (V-), U2.12 (V-)
Other:
- moved on the sheet: J2, R6, R8, R9, RV1, TP2, U1C
