File: Checkpoint 4/PWM/pcb_pwm/pcb_pwm.kicad_pcb (KiCad board)
At the start: 2 copper layers, 67 x 60.3 mm, 33 parts, among them J2 Conn_01x03_Socket, J3 Conn_01x06_Socket, U1 TL082, U2 LM2901

Commit message: sube cambios en el pcb del pwm, y cambios pruebas en la simu del buck
Parts:
- C3, C4: footprint Capacitor_THT:C_Disc_D5.0mm_W2.5mm_P5.00mm -> Capacitor_THT:C_Disc_D3.4mm_W2.1mm_P2.50mm
- D1: footprint Diode_THT:D_DO-27_P12.70mm_Horizontal -> Package_TO_SOT_THT:TO-220-2_Vertical
- R2: value 10k -> 500
- moved D1 12.9 mm to (170.5, 110.6)
Connections:
- C4 pad 1: -Vcc -> 0
- C4 pad 2: 0 -> -Vcc
- J3 pad 6: (no net) -> Vo
Routing:
- net Vo: track 76.7 -> 67.6 mm

Commit message: agrega ultimos cambios al pcb pwm?
Parts:
- moved D1 2.00 mm to (170.5, 108.6)
Routing:
- net Vo: track 67.6 -> 65.6 mm
Changed lines of the file:
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@@
 	(footprint "Package_TO_SOT_THT:TO-220-2_Vertical"
 		(layer "F.Cu")
-		(at 170.54 110.555 180)
+		(at 170.54 108.555 180)
 		(descr "TO-220-2, Vertical, RM 5.08mm, see https://www.centralsemi.com/PDFS/CASE/TO-220-2PD.PDF")
 		(tags "TO-220-2 Vertical RM 5.08mm")
@@
 		)
 	)
+	(gr_circle
+		(center 115.5 115)
+		(end 117.5 115)
+		(stroke
+			(width 0.2)
+			(type default)
+		)
+		(fill none)
+		(layer "B.Cu")
+	)
+	(gr_circle
+		(center 173 63)
+		(end 175 63)
+		(stroke
+			(width 0.2)
+			(type default)
+		)
+		(fill none)
+		(layer "B.Cu")
+	)
+	(gr_circle
+		(center 115 63)
+		(end 117 63)
+		(stroke
+			(width 0.2)
+			(type default)
+		)
+		(fill none)
+		(layer "B.Cu")
+	)
+	(gr_circle
+		(center 174 115.5)
+		(end 176 115.5)
+		(stroke
+			(width 0.2)
+			(type default)
+		)
+		(fill none)
+		(layer "B.Cu")
+	)
 	(gr_rect
 		(start 111 59.1)
@@
 	)
 	(segment
-		(start 172.2 76)
-		(end 165.3 76)
-		(width 1)
-		(layer "B.Cu")
-		(net 4)
-	)
-	(segment
 		(start 165.3 76)
 		(end 164.547057 76)
@@
 	)
 	(segment
-		(start 176.8 80.6)
-		(end 172.2 76)
-		(width 1)
-		(layer "B.Cu")
-		(net 4)
-	)
-	(segment
-		(start 170.54 110.555)
-		(end 170.54 106.96)
+		(start 172.2 76)
+		(end 165.3 76)
 		(width 1)
 		(layer "B.Cu")
@@
 	)
 	(segment
-		(start 176.8 100.7)
-		(end 176.8 80.6)
+		(start 176.8 80.6)
+		(end 172.2 76)
 		(width 1)
 		(layer "B.Cu")
@@
 	)
 	(segment
-		(start 170.54 106.96)
-		(end 176.8 100.7)
+		(start 170.54 108.555)
+		(end 170.54 106.96)
 		(width 1)
 		(layer "B.Cu")
@@
 	)
 	(segment
+		(start 170.54 106.96)
+		(end 176.8 100.7)
+		(width 1)
+		(layer "B.Cu")
+		(net 4)
+	)
+	(segment
 		(start 162.697057 77.85)
 		(end 163.934315 79.087258)
@@
 		(width 1)
 		(layer "B.Cu")
+		(net 4)
+	)
+	(segment
+		(start 176.8 100.7)
+		(end 176.8 80.6)
+		(width 1)
+		(layer "B.Cu")

Commit message: ahora está más lindo
Parts:
- moved D1 7.78 mm to (165.0, 114.1)
- moved RV1 4.70 mm to (142.5, 112.6)
Routing:
- net Vo: track 65.6 -> 73.4 mm
- net Net-(J2-Pin_3): track 22.2 -> 20.6 mm
Changed lines of the file:
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@@
 	(footprint "Package_TO_SOT_THT:TO-220-2_Vertical"
 		(layer "F.Cu")
-		(at 170.54 108.555 180)
+		(at 165.04 114.055 180)
 		(descr "TO-220-2, Vertical, RM 5.08mm, see https://www.centralsemi.com/PDFS/CASE/TO-220-2PD.PDF")
 		(tags "TO-220-2 Vertical RM 5.08mm")
@@
 	(footprint "Potentiometer_THT:Potentiometer_Piher_PC-16_Single_Horizontal"
 		(layer "F.Cu")
-		(at 147.2 112.6 -90)
+		(at 142.5 112.6 -90)
 		(descr "Potentiometer, horizontal, Piher PC-16 Single, http://www.piher-nacesa.com/pdf/20-PC16v03.pdf")
 		(tags "Potentiometer horizontal Piher PC-16 Single")
@@
 	)
 	(gr_circle
-		(center 115.5 115)
-		(end 117.5 115)
+		(center 116 114)
+		(end 118 114)
 		(stroke
 			(width 0.2)
@@
 	)
 	(gr_circle
-		(center 115 63)
-		(end 117 63)
+		(center 116 63)
+		(end 118 63)
 		(stroke
 			(width 0.2)
@@
 	)
 	(gr_circle
-		(center 174 115.5)
-		(end 176 115.5)
+		(center 173 114)
+		(end 175 114)
 		(stroke
 			(width 0.2)
@@
 	)
 	(segment
+		(start 176.8 80.6)
+		(end 172.2 76)
+		(width 1)
+		(layer "B.Cu")
+		(net 4)
+	)
+	(segment
+		(start 165.04 114.055)
+		(end 165.04 112.46)
+		(width 1)
+		(layer "B.Cu")
+		(net 4)
+	)
+	(segment
 		(start 165.3 76)
 		(end 164.547057 76)
@@
 	)
 	(segment
-		(start 176.8 80.6)
-		(end 172.2 76)
-		(width 1)
-		(layer "B.Cu")
-		(net 4)
-	)
-	(segment
 		(start 154.981371 77.781371)
 		(end 151.612742 81.15)
@@
 	)
 	(segment
-		(start 170.54 108.555)
-		(end 170.54 106.96)
+		(start 176.8 100.7)
+		(end 176.8 80.6)
 		(width 1)
 		(layer "B.Cu")
@@
 	)
 	(segment
-		(start 162.697057 77.85)
-		(end 155.05 77.85)
+		(start 165.04 112.46)
+		(end 176.8 100.7)
 		(width 1)
 		(layer "B.Cu")
@@
 	)
 	(segment
-		(start 170.54 106.96)
-		(end 176.8 100.7)
+		(start 162.697057 77.85)
+		(end 155.05 77.85)
 		(width 1)
 		(layer "B.Cu")
@@
 	)
 	(segment
-		(start 176.8 100.7)
-		(end 176.8 80.6)
-		(width 1)
-		(layer "B.Cu")
-		(net 4)
-	)
-	(segment
 		(start 118.9 94.537258)
 		(end 118.9 91.85)
@@
 	)
 	(segment
-		(start 141.74 104.3)
-		(end 141.74 108.99)
+		(start 141.74 103.097919)
+		(end 140.992081 102.35)
 		(width 1)
 		(layer "B.Cu")
@@
 	)
 	(segment
-		(start 141.74 108.99)
-		(end 144.17 111.42)
+		(start 141.74 103.097919)
+		(end 141.74 104.3)
 		(width 1)
 		(layer "B.Cu")
@@
 	)
 	(segment
-		(start 146.02 111.42)
-		(end 147.2 112.6)
+		(start 140 110.1)
+		(end 142.5 112.6)
 		(width 1)
 		(layer "B.Cu")
@@
 	)
 	(segment
-		(start 141.74 103.097919)
-		(end 140.992081 102.35)
+		(start 135.64 102.35)
+		(end 133.59 100.3)
 		(width 1)
 		(layer "B.Cu")
@@
 	)
 	(segment
-		(start 141.74 103.097919)
-		(end 141.74 104.3)
+		(start 141.74 106.26)
+		(end 140 108)
 		(width 1)
 		(layer "B.Cu")
@@
 	)
 	(segment
-		(start 135.64 102.35)
-		(end 133.59 100.3)
+		(start 140 108)
+		(end 140 110.1)
 		(width 1)
 		(layer "B.Cu")
@@
 	)
 	(segment
-		(start 144.17 111.42)
-		(end 146.02 111.42)
+		(start 140.992081 102.35)
+		(end 135.64 102.35)
 		(width 1)
 		(layer "B.Cu")
@@
 	)
 	(segment
-		(start 140.992081 102.35)
-		(end 135.64 102.35)
+		(start 141.74 104.3)
+		(end 141.74 106.26)
 		(width 1)
 		(layer "B.Cu")

Commit message: pcb pwm y buck final
Parts:
- C3, C4: footprint Capacitor_THT:C_Disc_D3.4mm_W2.1mm_P2.50mm -> Capacitor_THT:C_Disc_D4.3mm_W1.9mm_P5.00mm
- moved C4 4.99 mm to (147.2, 77.7), turned to 90 degrees
Connections:
- J3 pad 6: Vo -> unconnected-(J3-Pin_6-Pad6)
Routing:
- net Vref: track 44.0 -> 39.4 mm
- net Vcc: track 205.1 -> 201.1 mm
- net -Vcc: track 158.8 -> 155.4 mm
- net Vsin: track 63.3 -> 61.9 mm
Other:
- board size 67 x 60.3 mm -> 67.8 x 60.3 mm

Commit message: a ver si ahora si funcan los pcb sino me mato
Connections:
- R3 pad 2: Net-(U2A--) -> Net-(U2A-+)
- R4 pad 2: Net-(U2A--) -> Net-(U2A-+)
- U2 pad 4: Net-(U2A--) -> 0
- U2 pad 5: 0 -> Net-(U2A-+)
Routing:
- net Net-(U2A-+): track 0.00 -> 17.1 mm
- net Net-(U2A--): track 14.4 -> 0.00 mm
- net Vcc: track 201.1 -> 196.6 mm
- net Vsin: track 61.9 -> 59.7 mm
