File: Checkpoint 4/Support/pcb_support/pcb_support.kicad_pcb (KiCad board)
At the start: 2 copper layers, 29 parts, among them J1 Conn_01x03_Socket, U1 MC33063A-Q1_TRANS, U2 TL431, U6 TLV3201

Commit message: pcb support
Parts:
- moved C1 7.61 mm to (171.3, 111.0)
- moved TP3 6.51 mm to (170.8, 101.7)
- moved R12 5.19 mm to (175.8, 98.4)
Routing:
- net Net-(U6-IN+): track 17.2 -> 19.7 mm
- net Vbat: track 51.4 -> 53.5 mm
- net Vbuck: track 104.2 -> 105.8 mm
- net Venable: track 11.3 -> 10.4 mm
- added copper zone on B.Cu, net 0
Other:
- board outline added: 63.2 x 43 mm
