File: Checkpoint 4/Support/pcb_support/pcb_support.kicad_sch (KiCad schematic)
At the start: 29 parts, among them J1 Conn_01x03_Socket, U1 MC33063A-Q1_TRANS, U2 TL431, U6 TLV3201

Commit message: pcb support
Parts:
- renumbered C4 to C1, C5 to C2, C1 to C3, C2 to C4, C3 to C5, R11 to R1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
